File: GamerPCB.sch (KiCad schematic (older format))
At the start: 14 parts

Commit message: Initial PCB Design
Parts:
- added D1, D10, D11, D12, D13, D14, D15, D16, D17, D18, D19, D2, D3, D4, D5, D6, D7, D8, D9: D, Diode_SMD:D_SOD-123, symbol Device:D
- added F1: 500mA, Fuse:Fuse_1206_3216Metric, symbol Device:Polyfuse_Small
- added MX1, MX10, MX11, MX12, MX13, MX14, MX15, MX16, MX17, MX18, MX19, MX2, MX3, MX4, MX5, MX6, MX7, MX8, MX9: MX-LED, Kailh_Choc:KailhChoc-1U, symbol MX_Alps_Hybrid:MX-LED
- added R2, R3: 5.1k, Resistor_SMD:R_0805_2012Metric, symbol Device:R
- added USB1: HRO-TYPE-C-31-M-12, Type-C:HRO-TYPE-C-31-M-12-Assembly, symbol Type-C:HRO-TYPE-C-31-M-12
- C1, C2, C3, C4, C5, C6: renamed from C?; footprint (none) -> Capacitor_SMD:C_0805_2012Metric
- C7: renamed from C?; footprint (none) -> Diode_SMD:D_SOD-123
- R1, R4, R5, R6: renamed from R?; footprint (none) -> Resistor_SMD:R_0805_2012Metric
- SW1: renamed from SW?; footprint (none) -> random-keyboard-parts:SKQG-1155865
- Y1: renamed from Y?; footprint (none) -> Crystal:Crystal_SMD_3225-4Pin_3.2x2.5mm
- gave numbers to parts that had none: 1
Connections:
- net +5V: now also F1.1
- net D+: now also USB1.6 (DP1), USB1.8 (DP2)
- net D-: now also USB1.5 (DN2), USB1.7 (DN1)
- net GND: now also R2.2, R3.2, USB1.1 (GND), USB1.12 (GND)
- new net: R3.1, USB1.10 (CC2)
- new net: R2.1, USB1.4 (CC1)
- new net: D1.2 (A), MX1.2 (ROW)
- new net: D2.2 (A), MX2.2 (ROW)
- new net: D3.2 (A), MX3.2 (ROW)
- new net: D4.2 (A), MX4.2 (ROW)
- new net: D5.2 (A), MX5.2 (ROW)
- new net: D6.2 (A), MX6.2 (ROW)
- new net: D8.2 (A), MX8.2 (ROW)
- new net: D9.2 (A), MX9.2 (ROW)
- new net: D10.2 (A), MX10.2 (ROW)
- new net: D11.2 (A), MX11.2 (ROW)
- new net: D12.2 (A), MX12.2 (ROW)
- new net: D13.2 (A), MX13.2 (ROW)
- new net: D15.2 (A), MX15.2 (ROW)
- new net: D16.2 (A), MX16.2 (ROW)
- new net: D17.2 (A), MX17.2 (ROW)
- new net: D18.2 (A), MX18.2 (ROW)
- new net: D19.2 (A), MX19.2 (ROW)
- new net: D14.2 (A), MX14.2 (ROW)
- new net: D7.2 (A), MX7.2 (ROW)
- new net COL0: MX1.1 (COL), MX8.1 (COL)
- new net COL1: MX2.1 (COL), MX9.1 (COL)
- new net COL2: MX10.1 (COL), MX15.1 (COL), MX3.1 (COL)
- new net COL3: MX11.1 (COL), MX16.1 (COL), MX4.1 (COL)
- new net COL4: MX12.1 (COL), MX17.1 (COL), MX5.1 (COL)
- new net COL5: MX13.1 (COL), MX18.1 (COL), MX6.1 (COL)
- new net COL6: MX14.1 (COL), MX19.1 (COL), MX7.1 (COL)
- new net ROW0: D1.1 (K), D2.1 (K), D3.1 (K), D4.1 (K), D5.1 (K), D6.1 (K), D7.1 (K)
- new net ROW1: D10.1 (K), D11.1 (K), D12.1 (K), D13.1 (K), D14.1 (K), D8.1 (K), D9.1 (K)
- new net ROW2: D15.1 (K), D16.1 (K), D17.1 (K), D18.1 (K), D19.1 (K)
- new net VCC: F1.2, USB1.11 (VBUS), USB1.2 (VBUS)
Other:
- moved on the sheet: C1, C2, C3, C4, C5, C6, C7, R1, R4, R5, R6, SW1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
